File: Projects/Servo/boards/l0_servo/l0_servo.kicad_pcb (KiCad board)
At the start: 2 copper layers, 20.3 x 15.2 mm, 11 parts, among them J1 l0_Socket, Q1 NMOS_GSD, U1 LMV301

Commit message: change board kicad for project : Braekout board Luos Kit DC motor Servo
Parts:
- removed Q1: NMOS_GSD, Common_Footprint:SOT-23
- removed R1: 20k, Common_Footprint:R_0402_NoSilk
- removed R2, R4: 10k, Common_Footprint:R_0402_NoSilk
- removed R3: 68k, Common_Footprint:R_0402_NoSilk
- removed U1: LMV301, Common_Footprint:SC-70-5
- added D1: D_Zener, Common_Footprint:D_SOD-323F, F.Cu at (145.5, 65.9)
- added G***: LOGO, Common_Footprint:Luos_logo_xxsmall, F.Cu at (141.3, 66.2)
- renumbered S1 to s1, S2 to s2, S3 to s3, S4 to s4
Connections:
- J1 pad 10: /V_max -> Net-(J1-Pad10)
- J1 pad 12: /V_robus_img -> Net-(J1-Pad12)
- s1 pad 3: GNDREF -> GND
- s2 pad 3: GNDREF -> GND
- s3 pad 3: GNDREF -> GND
- s4 pad 3: GNDREF -> GND
Routing:
- net /V_robus_img: track 24.8 -> 0.00 mm, vias 2 -> 0
- net /V_max: track 16.0 -> 0.00 mm
- net VCC: track 38.7 -> 26.9 mm, vias 1 -> 0
- net GND: track 8.59 -> 0.00 mm, vias 2 -> 4
- net +3V3: track 7.01 -> 0.00 mm
- net Net-(R1-Pad2): track 3.27 -> 0.00 mm
- net Net-(J1-Pad1): track 10.4 -> 13.7 mm
- net Net-(J1-Pad9): track 22.7 -> 24.9 mm
- net Net-(J1-Pad8): track 20.2 -> 21.6 mm
- net Net-(J1-Pad4): track 8.38 -> 7.06 mm
- net GNDREF: vias 2 -> 0
- added copper zone on F.Cu, net GND
- removed copper zone on F.Cu, net GNDREF
Other:
- board text added: "Servo V0.0.2"
- board text removed: "Servo V0.0.1"
